Commit message: Implement Phase 1 3D perception and autonomous navigation stack

File: cstam-pkg/src/cstam_robot/urdf/cstam_robot.urdf.xacro (robot description, xacro)
@@ -4,8 +4,15 @@
   <xacro:arg name="robot_width" default="0.46"/>
   <xacro:arg name="chassis_height" default="0.20"/>
+  <xacro:arg name="base_clearance" default="0.025"/>
   <xacro:arg name="wheel_radius" default="0.075"/>
   <xacro:arg name="wheel_width" default="0.045"/>
+  <!-- Physical wheel-center spacing used to place the four wheels. -->
   <xacro:arg name="wheel_separation" default="0.41"/>
+  <!-- Empirically calibrated skid-steer track for Gazebo DiffDrive odometry. -->
+  <xacro:arg name="diff_drive_wheel_separation" default="0.455"/>
   <xacro:arg name="lidar_height" default="0.27"/>
+  <xacro:arg name="upper_lidar_height" default="0.82"/>
+  <xacro:arg name="lidar_3d_height" default="0.92"/>
+  <xacro:arg name="lidar_3d_x" default="0.24"/>
   <xacro:arg name="camera_height" default="1.12"/>
   <xacro:arg name="imu_height" default="0.72"/>
@@ -20,7 +27,9 @@
   <xacro:property name="robot_width" value="$(arg robot_width)"/>
   <xacro:property name="chassis_height" value="$(arg chassis_height)"/>
+  <xacro:property name="base_clearance" value="$(arg base_clearance)"/>
   <xacro:property name="wheel_radius" value="$(arg wheel_radius)"/>
   <xacro:property name="wheel_width" value="$(arg wheel_width)"/>
   <xacro:property name="wheel_separation" value="$(arg wheel_separation)"/>
+  <xacro:property name="diff_drive_wheel_separation" value="$(arg diff_drive_wheel_separation)"/>
   <xacro:property name="wheel_y" value="${wheel_separation / 2.0}"/>
   <xacro:cstam_base
@@ -28,4 +37,5 @@
     chassis_width="${robot_width - wheel_width}"
     chassis_height="${chassis_height}"
+    base_clearance="${base_clearance}"
     chassis_mass="8.0"
     wheel_radius="${wheel_radius}"
@@ -48,5 +58,9 @@
   <xacro:cstam_sensors
     chassis_height="${chassis_height}"
+    base_clearance="${base_clearance}"
     lidar_height="$(arg lidar_height)"
+    upper_lidar_height="$(arg upper_lidar_height)"
+    lidar_3d_height="$(arg lidar_3d_height)"
+    lidar_3d_x="$(arg lidar_3d_x)"
     camera_height="$(arg camera_height)"
     imu_height="$(arg imu_height)"
@@ -55,5 +69,5 @@
   <xacro:cstam_gazebo
     wheel_radius="${wheel_radius}"
-    wheel_separation="${wheel_separation}"
+    effective_wheel_separation="${diff_drive_wheel_separation}"
     max_linear_speed="0.8"/>
 </robot>

File: cstam-pkg/src/cstam_robot/urdf/cstam_robot_body.xacro (robot description, xacro)
@@ -4,5 +4,5 @@
                params="shelf_length shelf_width shelf_thickness shelf_1_z shelf_2_z shelf_3_z shelf_mass mast_z mast_height display_z">
     <link name="rear_panel_link">
-      <visual><geometry><box size="0.045 ${shelf_width} 0.83"/></geometry><material name="cstam_light_blue"/></visual>
+      <visual><visibility_flags>2</visibility_flags><geometry><box size="0.045 ${shelf_width} 0.83"/></geometry><material name="cstam_light_blue"/></visual>
       <collision><geometry><box size="0.045 ${shelf_width} 0.83"/></geometry></collision>
       <xacro:box_inertia mass="1.1" x="0.045" y="${shelf_width}" z="0.83"/>
@@ -14,5 +14,5 @@
     <!-- Full-height side supports keep all three delivery shelves attached. -->
     <link name="left_shelf_support_link">
-      <visual><geometry><box size="${shelf_length} 0.025 0.83"/></geometry><material name="cstam_light_blue"/></visual>
+      <visual><visibility_flags>2</visibility_flags><geometry><box size="${shelf_length} 0.025 0.83"/></geometry><material name="cstam_light_blue"/></visual>
       <collision><geometry><box size="${shelf_length} 0.025 0.83"/></geometry></collision>
       <xacro:box_inertia mass="0.35" x="${shelf_length}" y="0.025" z="0.83"/>
@@ -23,5 +23,5 @@
     </joint>
     <link name="right_shelf_support_link">
-      <visual><geometry><box size="${shelf_length} 0.025 0.83"/></geometry><material name="cstam_light_blue"/></visual>
+      <visual><visibility_flags>2</visibility_flags><geometry><box size="${shelf_length} 0.025 0.83"/></geometry><material name="cstam_light_blue"/></visual>
       <collision><geometry><box size="${shelf_length} 0.025 0.83"/></geometry></collision>
       <xacro:box_inertia mass="0.35" x="${shelf_length}" y="0.025" z="0.83"/>
@@ -33,5 +33,5 @@
     <!-- Each shelf is fixed to the rear panel, which is fixed to the chassis. -->
     <link name="shelf_1_link">
-      <visual><geometry><box size="${shelf_length} ${shelf_width} ${shelf_thickness}"/></geometry><material name="shelf_white"/></visual>
+      <visual><visibility_flags>2</visibility_flags><geometry><box size="${shelf_length} ${shelf_width} ${shelf_thickness}"/></geometry><material name="shelf_white"/></visual>
       <collision><geometry><box size="${shelf_length} ${shelf_width} ${shelf_thickness}"/></geometry></collision>
       <xacro:box_inertia mass="${shelf_mass}" x="${shelf_length}" y="${shelf_width}" z="${shelf_thickness}"/>
@@ -42,5 +42,5 @@
     </joint>
     <link name="shelf_2_link">
-      <visual><geometry><box size="${shelf_length} ${shelf_width} ${shelf_thickness}"/></geometry><material name="shelf_white"/></visual>
+      <visual><visibility_flags>2</visibility_flags><geometry><box size="${shelf_length} ${shelf_width} ${shelf_thickness}"/></geometry><material name="shelf_white"/></visual>
       <collision><geometry><box size="${shelf_length} ${shelf_width} ${shelf_thickness}"/></geometry></collision>
       <xacro:box_inertia mass="${shelf_mass}" x="${shelf_length}" y="${shelf_width}" z="${shelf_thickness}"/>
@@ -51,5 +51,5 @@
     </joint>
     <link name="shelf_3_link">
-      <visual><geometry><box size="${shelf_length} ${shelf_width} ${shelf_thickness}"/></geometry><material name="shelf_white"/></visual>
+      <visual><visibility_flags>2</visibility_flags><geometry><box size="${shelf_length} ${shelf_width} ${shelf_thickness}"/></geometry><material name="shelf_white"/></visual>
       <collision><geometry><box size="${shelf_length} ${shelf_width} ${shelf_thickness}"/></geometry></collision>
       <xacro:box_inertia mass="${shelf_mass}" x="${shelf_length}" y="${shelf_width}" z="${shelf_thickness}"/>
@@ -60,5 +60,5 @@
     </joint>
     <link name="sensor_mast_link">
-      <visual><geometry><box size="0.055 0.055 ${mast_height}"/></geometry><material name="cstam_blue"/></visual>
+      <visual><visibility_flags>2</visibility_flags><geometry><box size="0.055 0.055 ${mast_height}"/></geometry><material name="cstam_blue"/></visual>
       <collision><geometry><box size="0.055 0.055 ${mast_height}"/></geometry></collision>
       <xacro:box_inertia mass="0.45" x="0.055" y="0.055" z="${mast_height}"/>
@@ -69,5 +69,5 @@
     </joint>
     <link name="display_link">
-      <visual><geometry><box size="0.045 0.28 0.16"/></geometry><material name="display_green"/></visual>
+      <visual><visibility_flags>2</visibility_flags><geometry><box size="0.045 0.28 0.16"/></geometry><material name="display_green"/></visual>
       <collision><geometry><box size="0.045 0.28 0.16"/></geometry></collision>
       <xacro:box_inertia mass="0.35" x="0.045" y="0.28" z="0.16"/>

File: cstam-pkg/src/cstam_robot/urdf/cstam_robot_core.xacro (robot description, xacro)
@@ -2,17 +2,18 @@
 <robot xmlns:xacro="http://www.ros.org/wiki/xacro">
   <xacro:macro name="cstam_base"
-               params="chassis_length chassis_width chassis_height chassis_mass wheel_radius wheel_width wheel_y wheel_front_x wheel_rear_x wheel_mass">
+               params="chassis_length chassis_width chassis_height base_clearance chassis_mass wheel_radius wheel_width wheel_y wheel_front_x wheel_rear_x wheel_mass">
     <link name="base_footprint"/>
     <joint name="base_footprint_joint" type="fixed">
       <parent link="base_footprint"/>
       <child link="base_link"/>
-      <origin xyz="0 0 ${chassis_height / 2.0}" rpy="0 0 0"/>
+      <origin xyz="0 0 ${chassis_height / 2.0 + base_clearance}" rpy="0 0 0"/>
     </joint>
     <link name="base_link">
       <visual>
+        <visibility_flags>2</visibility_flags>
         <geometry><box size="${chassis_length} ${chassis_width} ${chassis_height}"/></geometry>
         <material name="cstam_blue"/>
       </visual>
-      <collision>
+      <collision name="base_link_collision">
         <geometry><box size="${chassis_length} ${chassis_width} ${chassis_height}"/></geometry>
       </collision>
@@ -23,4 +24,5 @@
       wheel_radius="${wheel_radius}"
       wheel_width="${wheel_width}"
+      base_clearance="${base_clearance}"
       wheel_y="${wheel_y}"
       wheel_front_x="${wheel_front_x}"

File: cstam-pkg/src/cstam_robot/urdf/cstam_robot_drivetrain.xacro (robot description, xacro)
@@ -2,17 +2,17 @@
 <robot xmlns:xacro="http://www.ros.org/wiki/xacro">
   <xacro:macro name="cstam_drivetrain"
-               params="chassis_height wheel_radius wheel_width wheel_y wheel_front_x wheel_rear_x wheel_mass">
+               params="chassis_height base_clearance wheel_radius wheel_width wheel_y wheel_front_x wheel_rear_x wheel_mass">
     <!-- Four-wheel skid-steer: one DiffDrive side controls two joints. -->
     <xacro:wheel name="left_front_wheel" x="${wheel_front_x}" y="${wheel_y}"
-                 z="${wheel_radius - chassis_height / 2.0}"
+                 z="${wheel_radius - chassis_height / 2.0 - base_clearance}"
                  radius="${wheel_radius}" width="${wheel_width}" mass="${wheel_mass}"/>
     <xacro:wheel name="left_rear_wheel" x="${wheel_rear_x}" y="${wheel_y}"
-                 z="${wheel_radius - chassis_height / 2.0}"
+                 z="${wheel_radius - chassis_height / 2.0 - base_clearance}"
                  radius="${wheel_radius}" width="${wheel_width}" mass="${wheel_mass}"/>
     <xacro:wheel name="right_front_wheel" x="${wheel_front_x}" y="${-wheel_y}"
-                 z="${wheel_radius - chassis_height / 2.0}"
+                 z="${wheel_radius - chassis_height / 2.0 - base_clearance}"
                  radius="${wheel_radius}" width="${wheel_width}" mass="${wheel_mass}"/>
     <xacro:wheel name="right_rear_wheel" x="${wheel_rear_x}" y="${-wheel_y}"
-                 z="${wheel_radius - chassis_height / 2.0}"
+                 z="${wheel_radius - chassis_height / 2.0 - base_clearance}"
                  radius="${wheel_radius}" width="${wheel_width}" mass="${wheel_mass}"/>
   </xacro:macro>
@@ -20,9 +20,10 @@
     <link name="${name}_link">
       <visual>
+        <visibility_flags>2</visibility_flags>
         <origin xyz="0 0 0" rpy="${pi / 2.0} 0 0"/>
         <geometry><cylinder radius="${radius}" length="${width}"/></geometry>
         <material name="rubber_black"/>
       </visual>
-      <collision>
+      <collision name="${name}_collision">
         <origin xyz="0 0 0" rpy="${pi / 2.0} 0 0"/>
         <geometry><cylinder radius="${radius}" length="${width}"/></geometry>

File: cstam-pkg/src/cstam_robot/urdf/cstam_robot_gazebo.xacro (robot description, xacro)
@@ -1,27 +1,81 @@
 <?xml version="1.0"?>
 <robot xmlns:xacro="http://www.ros.org/wiki/xacro">
-  <xacro:macro name="cstam_gazebo" params="wheel_radius wheel_separation max_linear_speed">
+  <xacro:macro name="cstam_gazebo" params="wheel_radius effective_wheel_separation max_linear_speed">
     <gazebo reference="base_link">
       <material>Gazebo/Blue</material>
+      <sensor name="base_contact" type="contact">
+        <always_on>true</always_on>
+        <update_rate>50</update_rate>
+        <topic>/cstam/contacts/base</topic>
+        <contact><collision>base_link_collision</collision></contact>
+      </sensor>
     </gazebo>
-    <gazebo reference="left_front_wheel_link"><mu1>1.1</mu1><mu2>0.8</mu2><material>Gazebo/Black</material></gazebo>
-    <gazebo reference="left_rear_wheel_link"><mu1>1.1</mu1><mu2>0.8</mu2><material>Gazebo/Black</material></gazebo>
-    <gazebo reference="right_front_wheel_link"><mu1>1.1</mu1><mu2>0.8</mu2><material>Gazebo/Black</material></gazebo>
-    <gazebo reference="right_rear_wheel_link"><mu1>1.1</mu1><mu2>0.8</mu2><material>Gazebo/Black</material></gazebo>
-    <gazebo reference="lidar_link">
-      <sensor name="cstam_lidar" type="gpu_lidar">
+    <gazebo reference="left_front_wheel_link">
+      <mu1>1.0</mu1><mu2>1.0</mu2><fdir1>1 0 0</fdir1>
+      <kp>1000000.0</kp><kd>10.0</kd><minDepth>0.001</minDepth>
+      <material>Gazebo/Black</material>
+      <sensor name="left_front_contact" type="contact">
+        <always_on>true</always_on><update_rate>50</update_rate>
+        <topic>/cstam/contacts/left_front</topic>
+        <contact><collision>left_front_wheel_collision</collision></contact>
+      </sensor>
+    </gazebo>
+    <gazebo reference="left_rear_wheel_link">
+      <mu1>1.0</mu1><mu2>1.0</mu2><fdir1>1 0 0</fdir1>
+      <kp>1000000.0</kp><kd>10.0</kd><minDepth>0.001</minDepth>
+      <material>Gazebo/Black</material>
+      <sensor name="left_rear_contact" type="contact">
+        <always_on>true</always_on><update_rate>50</update_rate>
+        <topic>/cstam/contacts/left_rear</topic>
+        <contact><collision>left_rear_wheel_collision</collision></contact>
+      </sensor>
+    </gazebo>
+    <gazebo reference="right_front_wheel_link">
+      <mu1>1.0</mu1><mu2>1.0</mu2><fdir1>1 0 0</fdir1>
+      <kp>1000000.0</kp><kd>10.0</kd><minDepth>0.001</minDepth>
+      <material>Gazebo/Black</material>
+      <sensor name="right_front_contact" type="contact">
+        <always_on>true</always_on><update_rate>50</update_rate>
+        <topic>/cstam/contacts/right_front</topic>
+        <contact><collision>right_front_wheel_collision</collision></contact>
+      </sensor>
+    </gazebo>
+    <gazebo reference="right_rear_wheel_link">
+      <mu1>1.0</mu1><mu2>1.0</mu2><fdir1>1 0 0</fdir1>
+      <kp>1000000.0</kp><kd>10.0</kd><minDepth>0.001</minDepth>
+      <material>Gazebo/Black</material>
+      <sensor name="right_rear_contact" type="contact">
+        <always_on>true</always_on><update_rate>50</update_rate>
+        <topic>/cstam/contacts/right_rear</topic>
+        <contact><collision>right_rear_wheel_collision</collision></contact>
+      </sensor>
+    </gazebo>
+    <!-- The legacy low and upper 2D LiDAR definitions are intentionally not
+         instantiated.  Their links and scan_self_filter remain available for
+         debugging, while the accepted Phase 1 runtime uses only cstam_3d_lidar. -->
+    <!-- One primary simulated 3D LiDAR.  Gazebo publishes a real
+         PointCloudPacked side topic at /lidar/points. -->
+    <gazebo reference="lidar_3d_link">
+      <sensor name="cstam_3d_lidar" type="gpu_lidar">
         <always_on>true</always_on>
         <visualize>true</visualize>
-        <update_rate>15</update_rate>
-        <topic>/scan</topic>
-        <gz_frame_id>lidar_link</gz_frame_id>
+        <update_rate>8</update_rate>
+        <topic>/lidar</topic>
+        <gz_frame_id>lidar_3d_link</gz_frame_id>
         <lidar>
+          <visibility_mask>1</visibility_mask>
           <scan>
             <horizontal>
-              <samples>720</samples>
+              <samples>360</samples>
               <resolution>1</resolution>
               <min_angle>-3.14159265</min_angle>
               <max_angle>3.14159265</max_angle>
             </horizontal>
+            <vertical>
+              <samples>16</samples>
+              <resolution>1</resolution>
+              <min_angle>-1.04719755</min_angle>
+              <max_angle>0.34906585</max_angle>
+            </vertical>
           </scan>
           <range>
@@ -54,7 +108,13 @@
         <right_joint>right_front_wheel_joint</right_joint>
         <right_joint>right_rear_wheel_joint</right_joint>
-        <wheel_separation>${wheel_separation}</wheel_separation>
+        <wheel_separation>${effective_wheel_separation}</wheel_separation>
         <wheel_radius>${wheel_radius}</wheel_radius>
         <max_velocity>${max_linear_speed}</max_velocity>
+        <max_linear_acceleration>1.0</max_linear_acceleration>
+        <min_linear_acceleration>-1.0</min_linear_acceleration>
+        <max_angular_acceleration>2.0</max_angular_acceleration>
+        <min_angular_acceleration>-2.0</min_angular_acceleration>
+        <max_angular_velocity>1.9</max_angular_velocity>
+        <min_angular_velocity>-1.9</min_angular_velocity>
         <odom_publish_frequency>30</odom_publish_frequency>
         <topic>/cmd_vel</topic>
@@ -62,5 +122,5 @@
         <tf_topic>/tf</tf_topic>
         <frame_id>odom</frame_id>
-        <child_frame_id>base_footprint</child_frame_id>
+        <child_frame_id>base_drive</child_frame_id>
       </plugin>
     </gazebo>

File: cstam-pkg/src/cstam_robot/urdf/cstam_robot_sensors.xacro (robot description, xacro)
@@ -1,8 +1,9 @@
 <?xml version="1.0"?>
 <robot xmlns:xacro="http://www.ros.org/wiki/xacro">
-  <xacro:macro name="cstam_sensors" params="chassis_height lidar_height camera_height imu_height mast_x mast_z">
+  <xacro:macro name="cstam_sensors" params="chassis_height base_clearance lidar_height upper_lidar_height lidar_3d_height lidar_3d_x camera_height imu_height mast_x mast_z">
     <!-- A visible pedestal connects the front LiDAR to the chassis. -->
     <link name="lidar_mount_link">
       <visual>
+        <visibility_flags>2</visibility_flags>
         <geometry><box size="0.06 0.09 0.05"/></geometry>
         <material name="cstam_blue"/>
@@ -17,5 +18,5 @@
     <!-- The LiDAR sits directly on the pedestal. -->
     <link name="lidar_link">
-      <visual><geometry><cylinder radius="0.055" length="0.045"/></geometry><material name="sensor_dark"/></visual>
+      <visual><visibility_flags>2</visibility_flags><geometry><cylinder radius="0.055" length="0.045"/></geometry><material name="sensor_dark"/></visual>
       <collision><geometry><cylinder radius="0.055" length="0.045"/></geometry></collision>
       <xacro:cylinder_inertia_y_axis mass="0.12" radius="0.055" length="0.045"/>
@@ -25,6 +26,27 @@
       <origin xyz="0 0 0.0475" rpy="0 0 0"/>
     </joint>
+    <!-- A second scan plane sees chair backs and table edges above the low
+         mapping LiDAR. Nav2 uses it locally; AMCL keeps the original scan. -->
+    <link name="lidar_upper_link"/>
+    <joint name="lidar_upper_joint" type="fixed">
+      <parent link="base_link"/><child link="lidar_upper_link"/>
+      <origin xyz="0.27 0 ${upper_lidar_height - chassis_height / 2.0 - base_clearance}" rpy="0 0 0"/>
+    </joint>
+    <!-- Primary Phase 1 multi-channel LiDAR mount. -->
+    <link name="lidar_3d_link">
+      <visual>
+        <visibility_flags>2</visibility_flags>
+        <geometry><cylinder radius="0.055" length="0.05"/></geometry>
+        <material name="sensor_dark"/>
+      </visual>
+      <collision><geometry><cylinder radius="0.055" length="0.05"/></geometry></collision>
+      <xacro:cylinder_inertia_y_axis mass="0.14" radius="0.055" length="0.05"/>
+    </link>
+    <joint name="lidar_3d_joint" type="fixed">
+      <parent link="base_link"/><child link="lidar_3d_link"/>
+      <origin xyz="${lidar_3d_x} 0 ${lidar_3d_height - chassis_height / 2.0 - base_clearance}" rpy="0 0 0"/>
+    </joint>
     <link name="camera_link">
-      <visual><geometry><box size="0.075 0.055 0.055"/></geometry><material name="sensor_dark"/></visual>
+      <visual><visibility_flags>2</visibility_flags><geometry><box size="0.075 0.055 0.055"/></geometry><material name="sensor_dark"/></visual>
       <collision><geometry><box size="0.075 0.055 0.055"/></geometry></collision>
       <xacro:box_inertia mass="0.10" x="0.075" y="0.055" z="0.055"/>
@@ -40,5 +62,5 @@
     </joint>
     <link name="imu_link">
-      <visual><geometry><box size="0.035 0.035 0.018"/></geometry><material name="sensor_dark"/></visual>
+      <visual><visibility_flags>2</visibility_flags><geometry><box size="0.035 0.035 0.018"/></geometry><material name="sensor_dark"/></visual>
       <xacro:box_inertia mass="0.04" x="0.035" y="0.035" z="0.018"/>
     </link>
@@ -57,5 +79,5 @@
   <xacro:macro name="ultrasonic_mount" params="name x y yaw">
     <link name="${name}_link">
-      <visual><geometry><cylinder radius="0.016" length="0.018"/></geometry><material name="ultrasonic_blue"/></visual>
+      <visual><visibility_flags>2</visibility_flags><geometry><cylinder radius="0.016" length="0.018"/></geometry><material name="ultrasonic_blue"/></visual>
       <collision><geometry><cylinder radius="0.016" length="0.018"/></geometry></collision>
       <xacro:cylinder_inertia_y_axis mass="0.015" radius="0.016" length="0.018"/>
