Commit message: Complete CSTAM Phase 1 autonomous delivery system

File: cstam-pkg/src/cstam_robot/urdf/cstam_robot.urdf.xacro (robot description, xacro)
@@ -10,5 +10,8 @@
   <xacro:arg name="wheel_separation" default="0.41"/>
   <!-- Empirically calibrated skid-steer track for Gazebo DiffDrive odometry. -->
-  <xacro:arg name="diff_drive_wheel_separation" default="0.455"/>
+  <!-- Pure-turn measurements at 0.15 rad/s: 1.5855/1.12921 and
+       3.1530/2.45609 rad (odom/physical). Least-squares correction of the
+       previous 0.455 m effective track gives approximately 0.60 m. -->
+  <xacro:arg name="diff_drive_wheel_separation" default="0.60"/>
   <xacro:arg name="lidar_height" default="0.27"/>
   <xacro:arg name="upper_lidar_height" default="0.82"/>

File: cstam-pkg/src/cstam_robot/urdf/cstam_robot_gazebo.xacro (robot description, xacro)
@@ -8,5 +8,27 @@
         <update_rate>50</update_rate>
         <topic>/cstam/contacts/base</topic>
-        <contact><collision>base_link_collision</collision></contact>
+        <!-- SDFormat conversion lumps the fixed base joint and renames the
+             collision. Contact sensors must reference the converted name. -->
+        <contact>
+          <collision>base_footprint_fixed_joint_lump__base_link_collision_collision</collision>
+          <collision>base_footprint_fixed_joint_lump__front_center_ultrasonic_link_collision_1</collision>
+          <collision>base_footprint_fixed_joint_lump__front_left_ultrasonic_link_collision_2</collision>
+          <collision>base_footprint_fixed_joint_lump__front_right_ultrasonic_link_collision_3</collision>
+          <collision>base_footprint_fixed_joint_lump__left_shelf_support_link_collision_4</collision>
+          <collision>base_footprint_fixed_joint_lump__lidar_3d_link_collision_5</collision>
+          <collision>base_footprint_fixed_joint_lump__lidar_mount_link_collision_6</collision>
+          <collision>base_footprint_fixed_joint_lump__lidar_link_collision_7</collision>
+          <collision>base_footprint_fixed_joint_lump__rear_center_ultrasonic_link_collision_8</collision>
+          <collision>base_footprint_fixed_joint_lump__rear_left_ultrasonic_link_collision_9</collision>
+          <collision>base_footprint_fixed_joint_lump__rear_panel_link_collision_10</collision>
+          <collision>base_footprint_fixed_joint_lump__shelf_1_link_collision_11</collision>
+          <collision>base_footprint_fixed_joint_lump__shelf_2_link_collision_12</collision>
+          <collision>base_footprint_fixed_joint_lump__shelf_3_link_collision_13</collision>
+          <collision>base_footprint_fixed_joint_lump__rear_right_ultrasonic_link_collision_14</collision>
+          <collision>base_footprint_fixed_joint_lump__right_shelf_support_link_collision_15</collision>
+          <collision>base_footprint_fixed_joint_lump__sensor_mast_link_collision_16</collision>
+          <collision>base_footprint_fixed_joint_lump__camera_link_collision_17</collision>
+          <collision>base_footprint_fixed_joint_lump__display_link_collision_18</collision>
+        </contact>
       </sensor>
     </gazebo>
@@ -18,5 +40,5 @@
         <always_on>true</always_on><update_rate>50</update_rate>
         <topic>/cstam/contacts/left_front</topic>
-        <contact><collision>left_front_wheel_collision</collision></contact>
+        <contact><collision>left_front_wheel_link_fixed_joint_lump__left_front_wheel_collision_collision</collision></contact>
       </sensor>
     </gazebo>
@@ -28,5 +50,5 @@
         <always_on>true</always_on><update_rate>50</update_rate>
         <topic>/cstam/contacts/left_rear</topic>
-        <contact><collision>left_rear_wheel_collision</collision></contact>
+        <contact><collision>left_rear_wheel_link_fixed_joint_lump__left_rear_wheel_collision_collision</collision></contact>
       </sensor>
     </gazebo>
@@ -38,5 +60,5 @@
         <always_on>true</always_on><update_rate>50</update_rate>
         <topic>/cstam/contacts/right_front</topic>
-        <contact><collision>right_front_wheel_collision</collision></contact>
+        <contact><collision>right_front_wheel_link_fixed_joint_lump__right_front_wheel_collision_collision</collision></contact>
       </sensor>
     </gazebo>
@@ -48,5 +70,5 @@
         <always_on>true</always_on><update_rate>50</update_rate>
         <topic>/cstam/contacts/right_rear</topic>
-        <contact><collision>right_rear_wheel_collision</collision></contact>
+        <contact><collision>right_rear_wheel_link_fixed_joint_lump__right_rear_wheel_collision_collision</collision></contact>
       </sensor>
     </gazebo>
@@ -103,4 +125,13 @@
     </gazebo>
     <gazebo>
+      <!-- Publish real wheel joint positions for RobotModel/TF visualization. -->
+      <plugin filename="gz-sim-joint-state-publisher-system"
+              name="gz::sim::systems::JointStatePublisher">
+        <topic>/joint_states</topic>
+        <joint_name>left_front_wheel_joint</joint_name>
+        <joint_name>left_rear_wheel_joint</joint_name>
+        <joint_name>right_front_wheel_joint</joint_name>
+        <joint_name>right_rear_wheel_joint</joint_name>
+      </plugin>
       <plugin filename="gz-sim-diff-drive-system" name="gz::sim::systems::DiffDrive">
         <left_joint>left_front_wheel_joint</left_joint>

File: cstam-pkg/src/cstam_robot/urdf/cstam_robot_sensors.xacro (robot description, xacro)
@@ -26,6 +26,6 @@
       <origin xyz="0 0 0.0475" rpy="0 0 0"/>
     </joint>
-    <!-- A second scan plane sees chair backs and table edges above the low
-         mapping LiDAR. Nav2 uses it locally; AMCL keeps the original scan. -->
+    <!-- Legacy upper scan frame retained for debugging. No runtime sensor
+         is attached here; Phase 1 uses the primary 3D LiDAR below. -->
     <link name="lidar_upper_link"/>
     <joint name="lidar_upper_joint" type="fixed">
